File: ecad/elec/layout/default/esp-box-emu.kicad_pcb (KiCad board)
At the start: 2 copper layers, 147.3 x 76.4 mm, 58 parts

Commit message: minor update
Other:
- board size 147.3 x 76.4 mm -> 72.5 x 76.4 mm
Changed lines of the file:
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@@
   (gr_arc (start 253.215 63.295) (mid 243.84 58.42) (end 248.715 49.045)
     (stroke (width 0.254) (type solid)) (layer "F.SilkS"))
+  (gr_line (start 62.5135 36.217) (end 62.5135 55.88)
+    (stroke (width 0.254) (type solid)) (layer "F.SilkS"))
   (gr_line (start 248.715 49.045) (end 262.685 44.845)
     (stroke (width 0.254) (type solid)) (layer "F.SilkS"))
@@
   (gr_arc (start 142.62 39.178) (mid 141.108772 38.852701) (end 139.87 37.928)
     (stroke (width 0.254) (type solid)) (layer "F.SilkS"))
-  (gr_circle (center 225.62 81.79) (end 227.32 81.79)
-    (stroke (width 0.1) (type solid)) (fill none) (layer "Edge.Cuts"))
   (gr_circle (center 137.721731 131.27906) (end 138.171731 131.27906)
     (stroke (width 0.2) (type solid)) (fill none) (layer "Edge.Cuts"))
@@
   (gr_line (start 186.8 126.11751) (end 186.8 71.120232)
     (stroke (width 0.2) (type solid)) (layer "Edge.Cuts"))
-  (gr_circle (center 257.62 113.79) (end 259.32 113.79)
-    (stroke (width 0.1) (type solid)) (fill none) (layer "Edge.Cuts"))
   (gr_circle (center 131.732269 130.448972) (end 132.182269 130.448972)
     (stroke (width 0.2) (type solid)) (fill none) (layer "Edge.Cuts"))
-  (gr_circle (center 257.62 81.79) (end 259.32 81.79)
-    (stroke (width 0.1) (type solid)) (fill none) (layer "Edge.Cuts"))
   (gr_arc (start 124.836 64.115881) (mid 124.255359 65.524941) (end 122.850569 66.11585)
     (stroke (width 0.2) (type solid)) (layer "Edge.Cuts"))
-  (gr_arc (start 261.62 113.79) (mid 260.448427 116.618427) (end 257.62 117.79)
-    (stroke (width 0.1) (type solid)) (layer "Edge.Cuts"))
   (gr_arc (start 118.076341 130.957951) (mid 115.355487 129.182592) (end 114.3 126.109991)
     (stroke (width 0.2) (type solid)) (layer "Edge.Cuts"))
@@
   (gr_circle (center 131.732269 130.448972) (end 132.182269 130.448972)
     (stroke (width 0.2) (type solid)) (fill none) (layer "Edge.Cuts"))
-  (gr_arc (start 225.62 117.79) (mid 222.791573 116.618427) (end 221.62 113.79)
-    (stroke (width 0.1) (type solid)) (layer "Edge.Cuts"))
   (gr_circle (center 133.495019 130.834822) (end 133.945019 130.834822)
     (stroke (width 0.2) (type solid)) (fill none) (layer "Edge.Cuts"))
@@
   (gr_circle (center 133.495019 130.834822) (end 133.945019 130.834822)
     (stroke (width 0.2) (type solid)) (fill none) (layer "Edge.Cuts"))
-  (gr_line (start 261.62 113.79) (end 261.62 81.79)
-    (stroke (width 0.1) (type solid)) (layer "Edge.Cuts"))
   (gr_line (start 114.3 71.12) (end 114.3 126.109991)
     (stroke (width 0.2) (type solid)) (layer "Edge.Cuts"))
-  (gr_line (start 221.62 81.79) (end 221.62 113.79)
-    (stroke (width 0.1) (type solid)) (layer "Edge.Cuts"))
   (gr_line (start 122.846447 66.119972) (end 119.299969 66.119972)
     (stroke (width 0.2) (type solid)) (layer "Edge.Cuts"))
-  (gr_arc (start 257.62 77.79) (mid 260.448427 78.961573) (end 261.62 81.79)
-    (stroke (width 0.1) (type solid)) (layer "Edge.Cuts"))
   (gr_arc (start 178.264 66.120241) (mid 176.849804 65.534452) (end 176.264 64.120241)
     (stroke (width 0.2) (type solid)) (layer "Edge.Cuts"))
   (gr_line (start 181.799991 66.120241) (end 178.264 66.120241)
     (stroke (width 0.2) (type solid)) (layer "Edge.Cuts"))
-  (gr_line (start 257.62 77.79) (end 225.62 77.79)
-    (stroke (width 0.1) (type solid)) (layer "Edge.Cuts"))
   (gr_line (start 122.850569 66.11585) (end 122.846447 66.119972)
     (stroke (width 0.2) (type solid)) (layer "Edge.Cuts"))
-  (gr_arc (start 221.62 81.79) (mid 222.791573 78.961573) (end 225.62 77.79)
-    (stroke (width 0.1) (type solid)) (layer "Edge.Cuts"))
   (gr_circle (center 127.546841 129.710972) (end 127.996841 129.710972)
     (stroke (width 0.2) (type solid)) (fill none) (layer "Edge.Cuts"))
-  (gr_circle (center 225.62 113.79) (end 227.32 113.79)
-    (stroke (width 0.1) (type solid)) (fill none) (layer "Edge.Cuts"))
   (gr_line (start 174.2642 58.616041) (end 126.823031 58.597091)
     (stroke (width 0.2) (type solid)) (layer "Edge.Cuts"))
   (gr_line (start 176.264 64.120241) (end 176.264 60.616041)
     (stroke (width 0.2) (type solid)) (layer "Edge.Cuts"))
-  (gr_line (start 225.62 117.79) (end 257.62 117.79)
-    (stroke (width 0.1) (type solid)) (layer "Edge.Cuts"))
   (gr_circle (center 137.721731 131.27906) (end 138.171731 131.27906)
     (stroke (width 0.2) (type solid)) (fill none) (layer "Edge.Cuts"))
@@
     (members
       3113d21e-59cc-4c0f-bee5-e833545d0b46
-      52866dd9-4755-400f-ba16-ad38915adcf8
-      541a1a79-62da-495c-9636-c14f351877f0
       5aa995c3-a63d-48ea-93dd-0369acd21e59
       8d29a89d-a9b5-44a4-a2ff-4f2fb64d7c47
-      929dbf3e-bebb-4297-b775-13c73b085766
-      f5bc7a96-627b-453a-a294-a1100af89213
     )
   )
@@
       3b51facc-3158-4d97-a9d8-3172536ac3a8
       43f505e9-4308-46ac-8850-967c5482321d
+      6cf1c938-585b-49f1-ae32-6091c681f835
       9cbf603d-5744-42f6-991d-917745b07d6c
       a3b40479-4bb6-4ec6-9bfa-d64b332df111
@@
     )
   )
-  (group "" (id deecda4f-8c94-4c72-8782-3da851560eb8)
-    (members
-      019c0a6d-9bb8-42f8-8584-8f200b71a27b
-      097c55d3-ce7a-4886-a7db-9a4e9fcd0127
-      0e8e5788-23b0-4e0e-993f-a94957498ae3
-      178364bc-250e-4a39-b0ba-4262bbac4b46
-      3d8baf97-c836-4397-867c-23e52ff05ce1
-      871dfad9-a85d-42ce-9d2d-6520fae7f4c4
-      8baef1cd-8e58-474a-b843-199aa0080763
-      a7e36be5-cc10-4aad-836f-bde309666136
-      b80e33ff-046b-4986-bc0d-6bc4865afc31
-      cf226ff4-3173-434d-8c9b-3129470c1ce4
-      d6648504-8f45-4127-8704-34acfec9c9a4
-      e1f36007-0f9d-4dc5-ae43-6b056652526f
-    )
-  )

Commit message: update headers (box) and layout
Parts:
- removed @HOLE10, @HOLE11 (x2), @HOLE9 (x2): , 
- added @HOLE0: , , F.Cu at (119.4, 71.2)
- added @HOLE1: , , F.Cu at (129.4, 70.7)
- added @HOLE2: , , F.Cu at (171.9, 70.7)
- added @HOLE3: , , F.Cu at (181.9, 71.2)
- added @HOLE4: , , F.Cu at (181.9, 126.2)
- added @HOLE5: , , F.Cu at (175.9, 126.2)
- added @HOLE6: , , F.Cu at (119.4, 126.2)
- added U$1: SILKSCREENGBC_D-PAD, GAMEBOY_COLOR_DPAD_SILK, F.Cu at (128.4, 90.5)
- added U$2: SILKSCREENGBC_START/SELECT, GAMEBOY_COLOR_START_SELECT_SILK, F.Cu at (149.8, 112.7)
- added U$3: SILKSCREENGBC_A/B, GAMEBOY_COLOR_A_B_BUTTON_MEMBRANE, F.Cu at (167.2, 82.9)
- added U$4: SILKSCREENGBC_A/B, GAMEBOY_COLOR_A_B_BUTTON_MEMBRANE, F.Cu at (172.4, 98.1)
- @HOLE7: moved to F.Cu
- U20, U21: footprint lib:HDR-TH_12P-P2.54-V-M-R2-C6-S2.54 -> lib:2X06_EDGE_REVERSED
- U22: footprint lib:HDR-TH_4P-P2.54-V-M-R2-C2-S2.54-1 -> lib:2X02_EDGE_REVERSED
- moved @HOLE7 78.0 mm to (125.4, 126.2), turned to 0 degrees
- moved R22 68.8 mm to (163.1, 68.6), turned to 180 degrees
- moved R23 61.9 mm to (163.6, 66.0), turned to 180 degrees
- moved LED1 55.0 mm to (150.0, 90.5)
- moved R9 48.7 mm to (154.4, 91.4)
- moved R8 41.4 mm to (141.7, 124.5)
- moved C1 7.26 mm to (122.7, 110.1)
- moved C2 7.26 mm to (122.7, 108.1)
- moved C3 7.26 mm to (122.6, 117.3)
- moved L1 7.26 mm to (126.9, 113.3)
- moved U3 7.26 mm to (123.2, 113.2)
- moved C4 7.26 mm to (122.6, 119.3)
- moved C5 7.26 mm to (119.8, 114.7)
- moved R5 7.26 mm to (123.3, 115.8)
- moved R6 7.26 mm to (121.4, 115.8)
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Routing:
- net cc2: track 1.65 -> 0.00 mm
- net cc1: track 1.60 -> 0.00 mm
- added copper zone on B.Cu, net 3V3
- added copper zone on B.Cu, net 5V
- added copper zone on F.Cu, net GND

Commit message: update pcb some more
Parts:
- moved R16 142.8 mm to (139.4, 73.7), turned to 180 degrees
- moved R17 136.8 mm to (144.3, 73.7), turned to 180 degrees
- moved R15 129.4 mm to (150.4, 73.7), turned to 180 degrees
- moved R14 123.6 mm to (155.3, 73.7), turned to 180 degrees
- moved U12 96.6 mm to (164.9, 99.9)
- moved U13 96.6 mm to (178.9, 95.0)
- moved U14 95.5 mm to (174.5, 79.9)
- moved U15 95.5 mm to (160.5, 84.9)
- moved R18 78.7 mm to (150.6, 119.4)
- moved U16 78.7 mm to (144.5, 112.7)
- moved U17 78.7 mm to (156.0, 112.7)
- moved R19 72.4 mm to (150.7, 121.9)
- moved R11 67.8 mm to (147.0, 92.9)
- moved R12 67.8 mm to (146.7, 87.8)
- moved R13 67.8 mm to (147.0, 80.2)
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