File: ecad/elec/layout/box-emu-base/box-emu-base.kicad_pcb (KiCad board)
At the start: 2 copper layers, 72.5 x 63.9 mm, 66 parts

Commit message: add net name overrides and update all boards
Connections:
- net a renamed drv2605.chip-a
- net b renamed drv2605.chip-b
- net p0_0 renamed up
- net p0_1 renamed down
- net p0_2 renamed left
- net p0_3 renamed right
- net p0_4 renamed io-a
- net p0_5 renamed io-b
- net p0_6 renamed x
- net p0_7 renamed y
- net p1_0 renamed start
- net p1_1 renamed select
- net p1_4 renamed vol_up
- net p1_5 renamed vol_down
