File: ecad/elec/layout/box-emu-base/box-emu-base.kicad_pcb (KiCad board)
At the start: 2 copper layers, 72.5 x 63.9 mm, 69 parts

Commit message: fix(ci): disable baked-in ATO_FROZEN and normalize base layout serialization
The atopile-kicad docker image sets ATO_FROZEN=1, silently forcing CI
builds into frozen mode, which fails on phantom in-memory diffs
(locked-attribute defaults, arc direction normalization) that never
reach the file on disk. Pass ATO_FROZEN=0 from the workflow — we verify
layout stability ourselves via canonicalize + git diff.

Also re-serialize box-emu-base.kicad_pcb through the same container
build + canonicalize pipeline CI runs: the file had last been written
by desktop KiCad (zone refills), whose s-expr dialect differs from
atopile's writer, so CI's rebuild produced an 8k-line formatting diff.
Verified idempotent across two container builds; DRC unchanged
(265 violations / 0 unconnected, same accepted classes).

Co-Authored-By: Claude Fable 5 <noreply@anthropic.com>
Parts:
- MECH1, MECH2: value SILKSCREENGBC_A/B -> (none)
- REF**: value BOX_EMU_BASE -> (none)
- U$1: value SILKSCREENGBC_D-PAD -> (none)
- U$2: value SILKSCREENGBC_START/SELECT -> (none)
