File: ecad/elec/layout/box-3-connector/box-3-connector.kicad_pcb (KiCad board)
At the start: 2 copper layers, 72.5 x 7.9 mm, 2 parts

Commit message: feat(ecad): Update ecad / atopile and improve workflow
Parts:
- removed U2: , lib:CONN-SMD_5-1734857-1
- added CN1: , TE_Connectivity_5_1734857_1:CONN-SMD_5-1734857-1, F.Cu at (0.29, 1.05)
- U1: footprint lib:BOX_3_EMU -> BOX_3_EMU_OUTLINE:BOX_3_EMU
- moved U1 168.0 mm to (0.00, 0.00)
