File: ecad/elec/layout/gbc-a-b-x-y/gbc-a-b-x-y.kicad_pcb (KiCad board)
At the start: 2 copper layers, 10 parts

Commit message: feat(ecad): Update ecad / atopile and improve workflow
Parts:
- removed U1, U4: , lib:GAMEBOY_COLOR_A_B_BUTTON_MEMBRANE
- removed U2, U3, U5, U6: , lib:GBC_A_B_BUTTON
- added MECH1: , GBC_A_B_MEMBRANE:GAMEBOY_COLOR_A_B_BUTTON_MEMBRANE, F.Cu at (0.00, 0.00)
- added MECH2: , GBC_A_B_MEMBRANE:GAMEBOY_COLOR_A_B_BUTTON_MEMBRANE, F.Cu at (30.0, 0.00)
- added SW1: , GBC_A_B_BUTTON:GBC_A_B_BUTTON, F.Cu at (10.0, 0.00)
- added SW2: , GBC_A_B_BUTTON:GBC_A_B_BUTTON, F.Cu at (20.0, 0.00)
- added SW3: , GBC_A_B_BUTTON:GBC_A_B_BUTTON, F.Cu at (40.0, 0.00)
- added SW4: , GBC_A_B_BUTTON:GBC_A_B_BUTTON, F.Cu at (50.0, 0.00)
- R1, R2, R3, R4: value 62.5mW Thick Film Resistors 50V ±100ppm/℃ ±1% 10kΩ 0402 Chip Resistor - Surface Mount ROHS -> 10kΩ ±1%; footprint lib:R0402 -> UNI_ROYAL_0402WGF1002TCE:R0402
- moved R2 161.0 mm to (30.0, -10.0), turned to 0 degrees
- moved R1 157.1 mm to (30.0, 0.00), turned to 0 degrees
- moved R4 154.1 mm to (60.0, -10.0), turned to 0 degrees
- moved R3 148.7 mm to (60.0, 0.00), turned to 0 degrees
Connections:
- net vcc renamed hv
- R1 pad 2: a -> line
- R2 pad 2: b -> b_btn-out-line
- R3 pad 2: x -> a-line
- R4 pad 2: y -> b-line
Routing:
- net gnd: track 46.0 -> 0.00 mm
- net y: track 28.3 -> 0.00 mm
- net b: track 28.3 -> 0.00 mm
- net x: track 13.7 -> 0.00 mm
- net a: track 13.7 -> 0.00 mm
Other:
- board text removed: "A"
- board text removed: "B"
- board text removed: "X"
- board text removed: "Y"
