File: ecad/elec/layout/gbc-a-b/gbc-a-b.kicad_pcb (KiCad board)
At the start: 2 copper layers, 5 parts

Commit message: feat(ecad): Update ecad / atopile and improve workflow
Parts:
- removed U1: , lib:GAMEBOY_COLOR_A_B_BUTTON_MEMBRANE
- removed U2, U3: , lib:GBC_A_B_BUTTON
- added MECH1: , GBC_A_B_MEMBRANE:GAMEBOY_COLOR_A_B_BUTTON_MEMBRANE, F.Cu at (0.00, 0.00)
- added SW1: , GBC_A_B_BUTTON:GBC_A_B_BUTTON, F.Cu at (10.0, 0.00)
- added SW2: , GBC_A_B_BUTTON:GBC_A_B_BUTTON, F.Cu at (20.0, 0.00)
- R1, R2: value 62.5mW Thick Film Resistors 50V ±100ppm/℃ ±1% 10kΩ 0402 Chip Resistor - Surface Mount ROHS -> 10kΩ ±1%; footprint lib:R0402 -> UNI_ROYAL_0402WGF1002TCE:R0402
- moved R2 140.4 mm to (30.0, -10.0), turned to 0 degrees
- moved R1 136.1 mm to (30.0, 0.00), turned to 0 degrees
Connections:
- net vcc renamed hv
- R1 pad 2: a -> contact_in
- R2 pad 2: b -> b_btn-out-contact_in
Routing:
- net b: track 28.3 -> 0.00 mm
- net gnd: track 23.0 -> 0.00 mm
- net a: track 13.7 -> 0.00 mm
Other:
- board text removed: "A"
- board text removed: "B"

Commit message: update to work with latest atopile services (lack thereof)
Parts:
- R1, R2: value 10kΩ ±1% -> 10kΩ ±5%
Changed lines of the file:
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@@
 			)
 		)
-		(property "Value" "10kΩ ±1%"
+		(property "Value" "10kΩ ±5%"
 			(at 0 4)
 			(layer "F.Fab")
@@
 			(hide yes)
 		)
-		(property "resistance" "10kΩ ±1%"
-			(at 0 0 0)
-			(layer "User.9")
-			(hide yes)
-		)
-		(property "max_power" "62.5mW"
-			(at 0 0 0)
-			(layer "User.9")
-			(hide yes)
-		)
-		(property "max_voltage" "50V"
+		(property "resistance" "10kΩ ±5%"
+			(at 0 0 0)
+			(layer "User.9")
+			(hide yes)
+		)
+		(property "max_power" "ℝ+W"
+			(at 0 0 0)
+			(layer "User.9")
+			(hide yes)
+		)
+		(property "max_voltage" "ℝ+V"
 			(at 0 0 0)
 			(layer "User.9")
@@
 			)
 		)
-		(property "Value" "10kΩ ±1%"
+		(property "Value" "10kΩ ±5%"
 			(at 0 4)
 			(layer "F.Fab")
@@
 			(hide yes)
 		)
-		(property "resistance" "10kΩ ±1%"
-			(at 0 0 0)
-			(layer "User.9")
-			(hide yes)
-		)
-		(property "max_power" "62.5mW"
-			(at 0 0 0)
-			(layer "User.9")
-			(hide yes)
-		)
-		(property "max_voltage" "50V"
-			(at 0 0 0)
-			(layer "User.9")
+		(property "resistance" "10kΩ ±5%"
+			(at 0 0 0)
+			(layer "User.9")
+			(hide yes)
+		)
+		(property "max_power" "ℝ+W"
+			(at 0 0 0)
+			(layer "User.9")
+			(hide yes)
+		)
+		(property "max_voltage" "ℝ+V"
+			(at 0 0 0)
+			(layer "User.9")
