File: ecad/elec/layout/box-connector/box-connector.kicad_pcb (KiCad board)
At the start: 2 copper layers, 72.5 x 12.5 mm, 4 parts

Commit message: feat(ecad): Update ECAD to support latest atopile and fix some bugs (#119)
* feat(ecad): Update ecad / atopile and improve workflow

* add step file to repo

* add box-3 step file

* improve workflow

* update the action to latest and fix some bugs / spurious issues

* remove legacy files

* update readme

* update deprecations

* improve placement of components and robustness of scripts

* nudge layouts some

* further layout changes

* fixing some issues

* fix broken ci

* minor update

* simple layout

* update to work with latest atopile services (lack thereof)

* update routing

* fix(ecad): vendor atopile registry package for CI builds

packages.atopileapi.com no longer resolves (taken down in the 0.16
platform migration, like the components API), so dependency resolution
of atopile/ti-tps63020@0.4.0 fails in CI and on any machine without a
warm .ato/modules. Commit the installed package (sans .cache) so
`ato build` finds it via its installed-package path and never contacts
the dead registry.

Co-Authored-By: Claude Fable 5 <noreply@anthropic.com>

* fix(ecad): keep vendored package byte-exact (no EOL normalization)

ato validates installed packages against the file hashes in
.package_meta.json; git's CRLF->LF normalization of the STEP files
changed their bytes on checkout, making CI fail with "Package has
local modifications". Exempt ecad/.ato/modules from text normalization
and re-commit the original bytes.

Co-Authored-By: Claude Fable 5 <noreply@anthropic.com>

* fix(ci): disable baked-in ATO_FROZEN and normalize base layout serialization

The atopile-kicad docker image sets ATO_FROZEN=1, silently forcing CI
builds into frozen mode, which fails on phantom in-memory diffs
(locked-attribute defaults, arc direction normalization) that never
reach the file on disk. Pass ATO_FROZEN=0 from the workflow — we verify
layout stability ourselves via canonicalize + git diff.

Also re-serialize box-emu-base.kicad_pcb through the same container
build + canonicalize pip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
Parts:
- removed U1: , lib:BOX_EMU
- removed U2, U3: , lib:2X06_EDGE_REVERSED
- added J1: , PMOD_2X06_EDGE:2X06_EDGE_REVERSED, F.Cu at (-7.10, 3.67)
- added J2: , PMOD_2X06_EDGE:2X06_EDGE_REVERSED, F.Cu at (15.8, 3.68)
- added REF**: , BOX_EMU_OUTLINE:BOX_EMU, F.Cu at (0.00, 0.00)
- U4: footprint lib:2X02_EDGE_REVERSED -> PWR_2X02_EDGE:2X02_EDGE_REVERSED; moved to B.Cu
- moved U4 180.6 mm to (-22.4, -2.68), turned to 180 degrees
Connections:
- net gnd renamed lv
- net pin2x2-_1 renamed power_5v-hv
